Commit message: Update meen_machine.urdf

File: ROS framework/urdf/meen_machine.urdf (robot description, URDF)
Before this commit: robot BlueRov2, 2 links, 1 joints
Joints:
- joint thruster_1_base_link: origin xyz=5.25 -4.26 -5.1 rpy=3.14 0 0 -> xyz=0.25 10.26 0.1 rpy=0 0 0; type continuous -> fixed

Commit message: Update meen_machine.urdf

File: ROS framework/urdf/meen_machine.urdf (robot description, URDF)
Before this commit: robot BlueRov2, 2 links, 1 joints
Joints:
- joint thruster_1_base_link: origin xyz=0.25 10.26 0.1 rpy=0 0 0 -> xyz=0.25 10.26 100 rpy=0 0 0

Commit message: Update meen_machine.urdf
thrusters are at proper position now

File: ROS framework/urdf/meen_machine.urdf (robot description, URDF)
Before this commit: robot BlueRov2, 2 links, 1 joints
Links:
- added link thruster_2; collision mesh filename=package://bluerov_ros_playground/meshes/T100.STL; visual mesh filename=package://bluerov_ros_playground/meshes/T100.STL
- added link thruster_3; collision mesh filename=package://bluerov_ros_playground/meshes/T100.STL; visual mesh filename=package://bluerov_ros_playground/meshes/T100.STL
- added link thruster_4; collision mesh filename=package://bluerov_ros_playground/meshes/T100.STL; visual mesh filename=package://bluerov_ros_playground/meshes/T100.STL
Joints:
- added joint thruster_2_base_link: type fixed, parent base_link, child thruster_2, origin xyz=-0.25 -10.26 100 rpy=0 0 0
- added joint thruster_3_base_link: type fixed, parent base_link, child thruster_3, origin xyz=0.25 10.26 100 rpy=0 0 0
- added joint thruster_4_base_link: type fixed, parent base_link, child thruster_4, origin xyz=0.25 -10.26 100 rpy=0 0 0
- joint thruster_1_base_link: origin xyz=0.25 10.26 100 rpy=0 0 0 -> xyz=-0.25 10.26 100 rpy=0 0 0
